File: HARDWARE/REV-J/_autosave-ESP32-EVB_Rev_I.sch (KiCad schematic (older format))
At the start: 148 parts, among them CON1 TB3 DG306-5.0-3P, CON2 TB3 DG306-5.0-3P, Q1 BC817-40(SOT23), Q2 BC817-40(SOT23), Q3 Q12MHz/20pF/30ppm/2P/HC-49SM(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, Q4 BC817-40(SOT23), Q5 BC817-40(SOT23), Q7 BC817-40(SOT23), U1 BL4054B-42TPRN(SOT23-5), U10 BAT54C(SOT23-3), U2 SY8089AAAC(SOT23-5), U3 ESP-WROOM-32, U4 LAN8710A-EZC(QFN32), U5 CH340T(SSOP20W), U6 MCP2562-E/SN(SOIC-8_150mil), U7 RPM7236-H8, U8 NCP303LSN27T1G(SOT-23-5), U9 BAT54C(SOT23-3)

Commit message: Update 434121043836 (rev1).stp, 5040771891.stp, and 173 more files...
Parts:
- added 5.0V/3.3V2: Closed(1-2)/Opened(2-3), OLIMEX_Jumpers-FP:SJ_2_SMALL_12_TIED, symbol ESP32-EVB_Rev_I:SJ2W_Closed(1-2)
- added R12, R13: 10k/R0603, OLIMEX_RLC-FP:R_0603_5MIL_DWS, symbol ESP32-EVB_Rev_I:R
Connections:
- net labels added: mb+
- wire segments 689 -> 690
Changed lines of the file:
@@
 	13900 13400 13900 13900
 Connection ~ 13900 13900
-Connection ~ 13700 13900
-Wire Wire Line
-	13000 13900 13700 13900
 Wire Wire Line
 	15600 13700 13000 13700
@@
 	13000 14000 15600 14000
 Wire Wire Line
-	13000 13800 13500 13800
-Wire Wire Line
-	13500 13800 13500 14900
+	13000 13800 13150 13800
 Wire Wire Line
 	19900 7800 18800 7800
@@
 Options: MCP2562-E/SN or SN65HVD232D usage!
 Wire Wire Line
-	12400 14000 11600 14000
-Wire Wire Line
-	11600 14000 11600 14400
-Wire Wire Line
-	11600 14400 12600 14400
-Wire Wire Line
 	2900 1800 2900 2100
 Wire Wire Line
@@
 Wire Wire Line
 	13700 13900 13700 14500
-$Comp
-L ESP32-EVB_Rev_I:+3.3V #PWR0101
-U 1 1 5B27C8D3
-P 12600 14400
-F 0 "#PWR0101" H 12600 14250 50  0001 C CNN
-F 1 "+3.3V" V 12600 14525 50  0000 L CNN
-F 2 "" H 12600 14400 60  0000 C CNN
-F 3 "" H 12600 14400 60  0000 C CNN
-	1    12600 14400
-	0    1    1    0
-$EndComp
 $Comp
 L ESP32-EVB_Rev_I:MCP2562-E_SN(SOIC-8_150mil) U6
@@
 	-1   0    0    1
 $EndComp
+Wire Wire Line
+	13000 13900 13150 13900
+Wire Wire Line
+	13150 13800 13150 13900
+Wire Wire Line
+	11500 13600 11800 13600
+Connection ~ 11500 13600
+Connection ~ 11800 13600
+$Comp
+L ESP32-EVB_Rev_I:R R12
+U 1 1 61A8BD6D
+P 10850 13800
+F 0 "R12" H 11025 13850 50  0000 C CNN
+F 1 "10k/R0603" H 10525 13850 50  0000 C CNN
+F 2 "OLIMEX_RLC-FP:R_0603_5MIL_DWS" V 10780 13800 30  0001 C CNN
+F 3 "" H 10850 13800 30  0000 C CNN
+	1    10850 13800
+	-1   0    0    -1
+$EndComp
+Connection ~ 11000 13800
+$Comp
+L ESP32-EVB_Rev_I:R R13
+U 1 1 61A8C506
+P 11650 14800
+F 0 "R13" H 11825 14850 50  0000 C CNN
+F 1 "10k/R0603" H 11325 14850 50  0000 C CNN
+F 2 "OLIMEX_RLC-FP:R_0603_5MIL_DWS" V 11580 14800 30  0001 C CNN
+F 3 "" H 11650 14800 30  0000 C CNN
+	1    11650 14800
+	-1   0    0    -1
+$EndComp
+Connection ~ 11500 14800
+$Comp
+L ESP32-EVB_Rev_I:GND #PWR0114
+U 1 1 61A8D549
+P 10700 13800
+F 0 "#PWR0114" H 10700 13550 50  0001 C CNN
+F 1 "GND" H 10700 13650 50  0000 C CNN
+F 2 "" H 10700 13800 60  0000 C CNN
+F 3 "" H 10700 13800 60  0000 C CNN
+	1    10700 13800
+	1    0    0    -1
+$EndComp
+Text Label 12250 13700 0    50   ~ 0
+mb+
+Text GLabel 11800 14800 2    50   Input ~ 0
+mb+
+$Comp
+L ESP32-EVB_Rev_I:+3.3V #PWR0101
+U 1 1 5B27C8D3
+P 12600 14200
+F 0 "#PWR0101" H 12600 14050 50  0001 C CNN
+F 1 "+3.3V" V 12600 14325 50  0000 L CNN
+F 2 "" H 12600 14200 60  0000 C CNN
+F 3 "" H 12600 14200 60  0000 C CNN
+	1    12600 14200
+	0    1    1    0
+$EndComp
+$Comp
+L ESP32-EVB_Rev_I:SJ2W_Closed(1-2) 5.0V/3.3V2
+U 1 1 61B60BDC
+P 12600 14400
+F 0 "5.0V/3.3V2" V 12900 14150 50  0000 L BNN
+F 1 "Closed(1-2)/Opened(2-3)" V 12800 13850 50  0000 L BNN
+F 2 "OLIMEX_Jumpers-FP:SJ_2_SMALL_12_TIED" H 12630 14550 20  0001 C CNN
+F 3 "" H 12600 14400 60  0000 C CNN
+	1    12600 14400
+	1    0    0    1
+$EndComp
+$Comp
+L ESP32-EVB_Rev_I:GND #PWR0115
+U 1 1 61C899C9
+P 12600 14600
+F 0 "#PWR0115" H 12600 14350 50  0001 C CNN
+F 1 "GND" H 12600 14450 50  0000 C CNN
+F 2 "" H 12600 14600 60  0000 C CNN
+F 3 "" H 12600 14600 60  0000 C CNN
+	1    12600 14600
+	1    0    0    -1
+$EndComp
+Wire Wire Line
+	12400 14400 11650 14400
+Wire Wire Line
+	11650 14400 11650 14000
+Wire Wire Line
+	11650 14000 12400 14000
 $EndSCHEMATC
