File: HARDWARE/REV-J/_autosave-ESP32-EVB_Rev_I.kicad_pcb (KiCad board)
At the start: 2 copper layers, 75.2 x 99.3 mm, 166 parts, among them CON1 TB3 DG306-5.0-3P, CON2 TB3 DG306-5.0-3P, Q1 BC817-40(SOT23), Q2 BC817-40(SOT23), Q3 Q12MHz/20pF/30ppm/2P/HC-49SM(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, Q4 BC817-40(SOT23), Q5 BC817-40(SOT23), Q6 BC817, Q7 BC817-40(SOT23), U1 BL4054B-42TPRN(SOT23-5), U10 BAT54C(SOT23-3), U2 SY8089AAAC(SOT23-5), U3 ESP-WROOM-32, U4 LAN8710A-EZC(QFN32), U5 CH340T(SSOP20W), U6 MCP2562-E/SN(SOIC-8_150mil), U7 RPM7236-H8, U8 NCP303LSN27T1G(SOT-23-5), U9 BAT54C(SOT23-3)

Commit message: Update ESP32-EVB_Rev_I.kicad_pcb, ESP32-EVB_Rev_I.kicad_pcb-bak, and _autosave-ESP32-EVB_Rev_I.kicad_pcb
Parts:
- moved MH3 0.72 mm to (73.3, 138.6)
Routing:
- net +3V3: track 243.8 -> 247.1 mm, vias 14 -> 15
- net Net-(BATT1-Pad1): track 72.4 -> 74.8 mm
- net Net-(U5-Pad7): track 52.0 -> 53.0 mm
- net Net-(U5-Pad6): track 48.2 -> 49.2 mm
- net GND: vias 134 -> 135
